File: 3DPrinter-PowerDistribution.sch (EAGLE design)
At the start: 74 parts, among them IC1 MAX31855K, IC2 MAX31855K, IC3 MAX31855K, IC4 EUP3476, J1 Extruder 1, J10 PCC-SMP-V-K, J11 Bed Heater, J12 PCC-SMP-V-K, J13 24V Input, J14 To Motor Drivers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

Commit message: foo
Parts:
- J2: value Fan 1 -> Mainboard; device con-wago-508:W237-02P -> con-harting:CON20L
- J3: value Mainboard -> Fan 1; device con-harting:CON16L -> con-wago-508:W237-02P; OC_FARNELL (none) -> unknown; OC_NEWARK (none) -> unknown
Connections:
- removed net EXTRUDER1_GATE: J3.3, R1.1, R5.1
- removed net EXTRUDER2_GATE: J3.4, R15.1, R20.1
- removed net X_LIMIT: J3.13, J6-3.S, LED1.C, R12.2
- removed net Y_LIMIT: J3.14, J7-3.S, LED2.C, R13.2
- removed net Z_LIMIT: J3.15, J8-3.S, LED3.C, R14.2
- new net E1_GATE: J2.3, R1.1, R5.1
- new net E2_GATE: J2.4, R15.1, R20.1
- new net X_MAX: J2.14
- new net X_MIN: J2.13, J6-3.S, LED1.C, R12.2
- new net Y_MAX: J2.16
- new net Y_MIN: J2.15, J7-3.S, LED2.C, R13.2
- new net Z_MAX: J2.18
- new net Z_MIN: J2.17, J8-3.S, LED3.C, R14.2
- net !TC1_CS: now also J2.8; no longer J3.8
- net !TC2_CS: now also J2.9; no longer J3.9
- net !TC3_CS: now also J2.10; no longer J3.10
- net +24V: now also J3-1.KL; no longer J2-1.KL
- net +3.3V: now also J2.19, J2.20; no longer J3.2
- net BEDHEATER_GATE: now also J2.5; no longer J3.5
- net FAN1_GATE: now also J2.6; no longer J3.6
- net FAN2_GATE: now also J2.7; no longer J3.7
- net GND: now also J2.1, J2.2; no longer J3.1, J3.16
- net MISO: now also J2.11; no longer J3.11
- net N$10: now also J3-2.KL; no longer J2-2.KL
- net SCK: now also J2.12; no longer J3.12
