File: 3DPrinter-PowerDistribution.brd (EAGLE design)
At the start: 86.4 x 31.8 mm, 30 parts, among them J1 Extruder 1, J2 24V Input, J3 To Motor Drivers, J4 To microcontroller board, J5 Extruder 2, J6 Bed Heater, Q1 PSMN1R3-30YL, Q2 PSMN1R3-30YL, Q3 PSMN1R3-30YL, Q4 PSMN1R3-30YL, Q5 PSMN1R3-30YL, Q6 PSMN1R3-30YL

Commit message: foo
Parts:
- removed SY5: OSHW-LOGOS, SparkFun:OSHW-LOGO-S
- added C1: 10nF, freetronics-master-v1:0603
- added C2: 22µF, freetronics-jon:C1206K
- added C3: 10µF, freetronics-jon:C1210K
- added C4: 2.2nF, freetronics-master-v1:0603
- added C5, C6, C7, C8: 100nF, freetronics-master-v1:0603
- added IC1, IC2, IC3: MAX31855K, RAMPSdisplay:MCLENG_SOIC-8
- added IC4: EUP3476, freetronics-luke:SO08T
- added J10, J12, J9: PCC-SMP-V-K, RAMPSdisplay:MCLAUGHLINENG_TC_JACK
- added J11: Bed Heater, con-wago-508:W237-132
- added J13: 24V Input, con-wago-508:W237-132
- added J14: To Motor Drivers, con-wago-508:W237-132
- added J7: Y Limit, con-molex:7395-03
- added J8: Z Limit, con-molex:7395-03
- added L1: 6.8 uH, freetronics-luke:CDRH
- added LED1: X Limit, freetronics-master-v1:LED-0603
- added LED2: Y Limit, freetronics-master-v1:LED-0603
- added LED3: Z Limit, freetronics-master-v1:LED-0603
- added LED4: Power, freetronics-master-v1:LED-0603
- added Q7: PSMN1R3-30YL, transistor-power:SOT669
- added R13, R14: 10kΩ, freetronics-master-v1:0603
- added R15, R20, R22, R29: 10Ω, freetronics-master-v1:0603
- added R16, R21, R23, R26, R30: 100kΩ, freetronics-master-v1:0603
- added R17, R18, R19: 10k, freetronics-master-v1:0603
- added R24: 1kΩ, freetronics-master-v1:0603
- added R25: 15k, freetronics-master-v1:0603
- added R27: 31k6, freetronics-master-v1:0603
- added R28: 10k 1%, freetronics-master-v1:0603
- added SY: OSHW-LOGOS, SparkFun:OSHW-LOGO-S
- J2: value 24V Input -> Fan 1
- J3: value To Motor Drivers -> Mainboard; device con-wago-508:W237-132 -> con-harting:CON16L
- J4: value To microcontroller board -> Fan 2; device con-molex:22-23-2051 -> con-wago-508:W237-132
- J6: value Bed Heater -> X Limit; device con-wago-508:W237-132 -> con-molex:7395-03
- Q2: value PSMN1R3-30YL -> FDS9926; device transistor-power:SOT669 -> zetex:SM8
- R10, R8: value 100kΩ -> 1kΩ
- R11: value 10Ω -> 100kΩ
- R12: value 100kΩ -> 10kΩ
- R9: value 10Ω -> 1kΩ
- moved J3 74.0 mm to (100.3, 26.7), turned to 270 degrees
- moved J2 69.9 mm to (85.1, 6.35)
- moved J6 56.8 mm to (34.3, 49.5), turned to 180 degrees
- moved Q2 50.8 mm to (90.2, 17.8)
- moved H4 43.3 mm to (109.2, 59.7)
- moved J4 36.3 mm to (99.1, 6.35), turned to 0 degrees
- moved R3 35.5 mm to (72.4, 31.8), turned to 0 degrees
- moved R4 33.1 mm to (67.3, 31.8), turned to 0 degrees
- moved H2 33.0 mm to (5.08, 59.7)
- moved R8 31.5 mm to (80.0, 30.5), turned to 0 degrees
- moved H3 27.9 mm to (109.2, 5.08)
- moved R7 23.7 mm to (67.3, 40.6), turned to 0 degrees
- moved Q3 21.6 mm to (39.4, 16.5)
- moved Q5 21.6 mm to (53.3, 16.5)
- moved R12 19.6 mm to (80.0, 33.0), turned to 0 degrees
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Connections:
- new net !TC1_CS: IC1.CS, J3.8, R17.2
- new net !TC2_CS: IC2.CS, J3.9, R18.2
- new net !TC3_CS: IC3.CS, J3.10, R19.2
- new net +3.3V: C2.1, C6.1, C7.1, C8.1, IC1.VCC, IC2.VCC, IC3.VCC, J3.2, J6.1, J7.1, J8.1, L1.2, R10.1, R12.1, R13.1, R14.1, R17.1, R18.1, R19.1, R24.1, R27.1, R8.1, R9.1
- new net BEDHEATER_GATE: J3.5, R22.1, R29.1
- new net EXTRUDER1_GATE: J3.3, R1.1, R5.1
- new net EXTRUDER2_GATE: J3.4, R15.1, R20.1
- new net FAN1_GATE: J3.6, R3.1
- new net FAN2_GATE: J3.7, R7.1
- new net MISO: IC1.SO, IC2.SO, IC3.SO, J3.11
- new net N$10: J2.2, Q2.5
- new net N$12: J4.2, Q2.7
- new net N$15: LED1.A, R8.2
- new net N$16: LED2.A, R9.2
- new net N$17: LED3.A, R10.2
- new net N$21: LED4.A, R24.2
- new net N$28: IC3.T-, J12.T-
- new net N$29: IC3.T+, J12.T+
- new net N$3: Q4.4, R15.2, R16.1
- new net N$32: IC2.T-, J10.T-
- new net N$33: IC2.T+, J10.T+
- new net N$42: IC4.7, R23.1
- new net N$44: C1.1, IC4.3, L1.1
- new net N$51: C1.2, IC4.1
- new net N$59: C4.2, R25.2
- new net N$61: IC4.6, R25.1
- new net N$62: C5.2, IC4.8
- new net N$63: IC4.5, R27.2, R28.1
- new net SCK: IC1.SCK, IC2.SCK, IC3.SCK, J3.12
- new net X_LIMIT: J3.13, J6.3, LED1.C, R12.2
- new net Y_LIMIT: J3.14, J7.3, LED2.C, R13.2
- new net Z_LIMIT: J3.15, J8.3, LED3.C, R14.2
- net +24V: now also C3.1, IC4.2, J11.1, J14.1, J2.1, J4.1, R23.2; no longer J3.1, J4.4, J6.1
- net GND: now also C2.2, C3.2, C4.1, C5.1, C6.2, C7.2, C8.2, IC1.GND, IC2.GND, IC3.GND, IC4.4, IC4.9, J10.P$1, J10.P$2, J12.P$1, J12.P$2, J13.2, J14.2, J3.1, J3.16, J6.2, J7.2, J8.2, J9.P$1, J9.P$2, LED4.C, Q7.1, Q7.2, Q7.3, R11.2, R16.2, R21.2, R26.2, R28.2, R30.2; no longer J2.2, J3.2, J4.5, Q2.2, R10.2, R12.2, R8.2
- net J5: now also J11.2, Q7.MB; no longer J6.2, Q5.MB
- net N$11: now also IC1.T-, J9.T-; no longer J4.2, R5.1, R7.1
- net N$14: now also Q2.2, R11.1, R7.2; no longer J4.3, R1.1, R3.1
- net N$2: now also Q3.MB; no longer Q2.MB
- net N$4: now also Q5.MB; no longer Q3.MB
- net N$5: now also Q5.4, R20.2, R21.1; no longer Q4.4, R7.2, R8.1
- net N$6: now also J13.1; no longer J2.1
- net N$7: now also Q6.4, R22.2, R26.1; no longer Q5.4, R10.1, R9.2
- net N$8: now also IC1.T+, J9.T+; no longer J4.1, R11.1, R9.1
- net N$9: now also Q7.4, R29.2, R30.1; no longer Q6.4, R11.2, R12.1
Routing:
- net N$14: track 39.5 -> 0.00 mm, vias 2 -> 0
- net +3.3V: track 0.00 -> 37.6 mm
- net MISO: track 0.00 -> 28.6 mm
- net SCK: track 0.00 -> 24.1 mm, vias 0 -> 3
- net N$11: track 28.5 -> 8.26 mm, vias 2 -> 0
- net N$12: track 0.00 -> 16.7 mm
- net N$29: track 0.00 -> 13.8 mm
- net N$33: track 0.00 -> 13.8 mm
- net N$44: track 0.00 -> 11.1 mm
- net BEDHEATER_GATE: track 0.00 -> 10.5 mm, vias 0 -> 2
- net EXTRUDER2_GATE: track 0.00 -> 10.5 mm, vias 0 -> 2
- net N$10: track 0.00 -> 9.07 mm
- net EXTRUDER1_GATE: track 0.00 -> 7.19 mm, vias 0 -> 2
- net N$13: track 5.42 -> 0.00 mm
- net N$3: track 0.00 -> 5.42 mm
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Other:
- board size 86.4 x 31.8 mm -> 114.3 x 64.8 mm

Commit message: foo
Parts:
- J2: value Fan 1 -> Mainboard; device con-wago-508:W237-132 -> con-harting:CON20L
- J3: value Mainboard -> Fan 1; device con-harting:CON16L -> con-wago-508:W237-132
- moved H2 101.0 mm to (102.9, 34.3)
- moved J2 47.1 mm to (73.7, 52.1)
- moved J3 25.4 mm to (85.1, 6.35), turned to 0 degrees
- moved H4 7.62 mm to (109.2, 52.1)
Connections:
- removed net EXTRUDER1_GATE: J3.3, R1.1, R5.1
- removed net EXTRUDER2_GATE: J3.4, R15.1, R20.1
- removed net X_LIMIT: J3.13, J6.3, LED1.C, R12.2
- removed net Y_LIMIT: J3.14, J7.3, LED2.C, R13.2
- removed net Z_LIMIT: J3.15, J8.3, LED3.C, R14.2
- new net E1_GATE: J2.3, R1.1, R5.1
- new net E2_GATE: J2.4, R15.1, R20.1
- new net X_MAX: J2.14
- new net X_MIN: J2.13, J6.3, LED1.C, R12.2
- new net Y_MAX: J2.16
- new net Y_MIN: J2.15, J7.3, LED2.C, R13.2
- new net Z_MAX: J2.18
- new net Z_MIN: J2.17, J8.3, LED3.C, R14.2
- net !TC1_CS: now also J2.8; no longer J3.8
- net !TC2_CS: now also J2.9; no longer J3.9
- net !TC3_CS: now also J2.10; no longer J3.10
- net +24V: now also J3.1; no longer J2.1
- net +3.3V: now also J2.19, J2.20; no longer J3.2
- net BEDHEATER_GATE: now also J2.5; no longer J3.5
- net FAN1_GATE: now also J2.6; no longer J3.6
- net FAN2_GATE: now also J2.7; no longer J3.7
- net GND: now also J2.1, J2.2; no longer J3.1, J3.16
- net MISO: now also J2.11; no longer J3.11
- net N$10: now also J3.2; no longer J2.2
- net SCK: now also J2.12; no longer J3.12
Routing:
- net EXTRUDER2_GATE: track 10.5 -> 0.00 mm, vias 2 -> 0
- net E2_GATE: track 0.00 -> 10.5 mm, vias 0 -> 2
- net EXTRUDER1_GATE: track 7.19 -> 0.00 mm, vias 2 -> 0
- net E1_GATE: track 0.00 -> 7.19 mm, vias 0 -> 2
Other:
- board size 114.3 x 64.8 mm -> 114.3 x 57.1 mm
