File: 3DPrinter-mainboard.sch (EAGLE design)
At the start: 18 parts, among them J10 Touchscreen, J11 Touchscreen, J31 Power Board, J58 Stepper Driver Board, J6 MicroSD Card

Commit message: foo
Parts:
- removed H1, H2, H3, H4: HOLE, holes:MOUNT-HOLE3.2
- removed J10: Touchscreen, pinhead:PINHD-1X4
- removed J11: Touchscreen, SparkFun:DS_TOUCH_CONNECTOR
- removed J31: Power Board, con-harting:CON16L
- removed J58: Stepper Driver Board, con-harting:CON20L
- added C10, C11, C3, C5, C6, C7: 100nF, freetronics-master-v1:CAP0603
- added C12: 4.7µF, freetronics-master-v1:CAP0805
- added C2, C4: 22pF, freetronics-master-v1:CAP0603
- added C8, C9: 47pF, freetronics-master-v1:CAP0603
- added F1: 500mA, freetronics-luke:PTC
- added IC1: TL331, linear:TL331
- added IC2: ATMEGA2560-16AU, atmel-2005:ATMEGA1280-16AU
- added IC3: FT230X, serial:FT230XQ
- added J1: Encoder, con-molex:22-05-7048-04
- added J2: Power Board, con-harting:CON20L
- added J3: MicroSD Card, RAMPSdisplay:ADAFRUIT_MICROSD
- added J4: ISP, freetronics-master-v1:PINHD-2X3
- added J5: I2C, freetronics-master-v1:M02PTH
- added LED2: Rx/Grn, freetronics-master-v1:LED0603
- added LED3: Tx/Yel, freetronics-master-v1:LED0603
- added Q1: 16MHz, freetronics-master-v1:CRYSTALHC49US
- added Q2: Piezo, RAMPSdisplay:FREETRONICS-MASTER-V1_BUZZERSMD12X12
- added Q3: 2N7002, freetronics-master-v1:MOSFET-NCHANNELSMD
- added R10, R14, R15: 1kΩ, freetronics-master-v1:RESISTOR0603
- added R11: 22Ω, freetronics-master-v1:RESISTOR0603
- added R13, R16: 27Ω, freetronics-master-v1:RESISTOR0603
- added R4, R5, R7, R8, R9: 10kΩ, freetronics-master-v1:RESISTOR0603
- added R6: 3.3kΩ, freetronics-master-v1:RESISTOR0603
- added S1: Reset, SparkFun:SWITCH-MOMENTARY-2SMD
- added X1: USB-MICROB, freetronics-master-v1:USB-MICROB
- J6: value MicroSD Card -> Stepper Driver Board; device RAMPSdisplay:ADAFRUIT_MICROSD -> con-harting:CON26L
- R12: value 22Ω -> 10kΩ
- R3: value 1kΩ -> 10kΩ
Connections:
- removed net +3.3V: J31.2
- removed net EXTRUDER1_GATE: J31.3
- removed net EXTRUDER2_GATE: J31.4
- removed net LCD_E: LCD1.E
- removed net N$59: LCD1.BA, R12.1
- removed net TOUCH1: J10.1, J11.Y1
- removed net TOUCH2: J10.2, J11.X2
- removed net TOUCH3: J10.3, J11.Y2
- removed net TOUCH4: J10.4, J11.X1
- removed net VDD: C1.1, J6.VDD
- removed net X_LIMIT: J31.13
- removed net Y_LIMIT: J31.14
- removed net Z_LIMIT: J31.15
- new net !RESET: C1.2, IC2.RESET, J4.5, R5.2, S1.2
- new net +5V: C11.1, C12.1, F1.P$2, IC3.RESET#, IC3.VCC
- new net BUZZER: IC1.V+, IC2.(A12)PC4
- new net CTS: C1.1, IC3.CTS#
- new net E1_ENABLE: IC2.(AD2)PA2, J6.21
- new net E1_GATE: IC2.PH5(OC4C), J2.3
- new net E2_ENABLE: IC2.(A15)PC7, J6.22
- new net E2_GATE: IC2.PH6(OC2B), J2.4
- new net ENCODER_A: IC2.(A10)PC2, J1-1.S, R1.2
- new net ENCODER_B: IC2.(A8)PC0, J1-2.S, R2.2
- new net ENCODER_SWITCH: IC2.(AD0)PA0, J1-3.S, R3.2
- new net LCD_BL: IC2.(OC0A/OC1C/PCINT7)PB7, Q3.G, R12.2
- new net LCD_EN: IC2.PH0(RXD2), LCD1.E
- new net N$1: LCD1.BK, R11.1
- new net N$10: IC3.CBUS1, R15.2
- new net N$11: LED2.C, R14.1
- new net N$12: IC3.CBUS2, R14.2
- new net N$2: LED3.C, R15.1
- new net N$3: Q3.D, R11.2
- new net N$30: C3.1, IC1.-IN, R6.2
- new net N$31: IC1.+IN, R4.2, R7.2
- new net N$34: IC1.OUT, Q2.2, R4.1, R6.1
- new net N$36: C4.2, IC2.XTAL1, Q1.1
- new net N$37: C10.1, IC3.3V3OUT, IC3.VCCIO
- new net N$38: C6.1, IC2.AREF
- new net N$39: IC3.USBDP, R16.1
- new net N$4: IC3.USBDM, R13.1
- new net N$40: C8.1, R16.2, X1.D+
- new net N$41: C9.1, R13.2, X1.D-
- new net N$52: F1.P$1, X1.VBUS
- new net N$8: C2.2, IC2.XTAL2, Q1.2
- new net RXD0: IC2.(RXD0/PCIN8)PE0, IC3.TXD
- new net SCL: IC2.(SCL/INT0)PD0, J5.2
- new net SDA: IC2.(SDA/INT1)PD1, J5.1
- new net TXD0: IC2.(TXD0)PE1, IC3.RXD
- new net X_ENABLE: IC2.(T0)PD7, J6.18
- new net X_MAX: IC2.(OC3B/INT4)PE4, J2.14
- new net X_MIN: IC2.(OC3C/INT5)PE5, J2.13
- new net Y_ENABLE: IC2.(OC1A/PCINT5)PB5, J6.19
- new net Y_MAX: IC2.PJ0(RXD3/PCINT9), J2.16
- new net Y_MIN: IC2.PJ1(TXD3/PCINT10), J2.15
- new net Z_ENABLE: IC2.(OC1B/PCINT6)PB6, J6.20
- new net Z_MAX: IC2.(RXD1/INT2)PD2, J2.18
- new net Z_MIN: IC2.(TXD1/INT3)PD3, J2.17
- net !SD_CS: now also IC2.PL7, J3.CS, R10.2, R8.2; no longer J6.CS, R2.2, R3.2
- net !SD_DETECT: now also IC2.(WR)PG0, J3.CARD_DETECT, R9.2; no longer J6.CARD_DETECT, R1.2
- net !TC1_CS: now also IC2.PL6, J2.8; no longer J31.8
- net !TC2_CS: now also IC2.PL5(OC5C), J2.9; no longer J31.9
- net !TC3_CS: now also IC2.PL4(OC5B), J2.10; no longer J31.10
- net +24V: now also J6.24, J6.26; no longer J58.20
- net +3V3: now also C5.1, C7.1, IC2.AVCC, IC2.VCC, IC2.VCC1, IC2.VCC2, IC2.VCC3, J2.19, J2.20, J3.VDD, J4.2, J6.23, J6.25, LCD1.BA, LED2.A, LED3.A, R12.1, R3.1, R5.1, R8.1, R9.1; no longer J58.18, J58.2, R12.2
- net BEDHEATER_GATE: now also IC2.(OC2A/PCINT4)PB4, J2.5; no longer J31.5
- net E1_DIR: now also IC2.(AD6)PA6, J6.9; no longer J58.10
- net E1_STEP: now also IC2.(AD4)PA4, J6.10; no longer J58.9
- net E1_VREF: now also IC2.(ADC3)PF3, J6.16; no longer J58.16
- net E2_DIR: now also IC2.(A11)PC3, J6.11; no longer J58.12
- net E2_STEP: now also IC2.(A9)PC1, J6.12; no longer J58.11
- net E2_VREF: now also IC2.(ADC4/TCK)PF4, J6.17; no longer J58.17
- net FAN1_GATE: now also IC2.(ALE)PG2, J2.6; no longer J31.6
- net FAN2_GATE: now also IC2.(RD)PG1, J2.7; no longer J31.7
- net GND: now also C10.2, C11.2, C12.2, C2.1, C3.2, C4.1, C5.2, C6.2, C7.2, C8.2, C9.2, IC1.GND, IC2.AGND, IC2.GND, IC2.GND1, IC2.GND2, IC2.GND3, IC3.GND1, IC3.GND2, IC3.GND3, J1-4.S, J2.1, J2.2, J3.GND, J3.GND1, J3.VSS, J4.6, J6.1, J6.2, Q2.1, Q3.S, R7.1, S1.1, X1.GND; no longer C1.2, J31.1, J31.16, J58.1, J58.19, J6.GND, J6.GND1, J6.VSS, LCD1.BK
- net LCD_D4: now also IC2.(AD1)PA1
- net LCD_D5: now also IC2.(AD3)PA3
- net LCD_D6: now also IC2.(AD5)PA5
- net LCD_D7: now also IC2.(AD7)PA7
- net LCD_RS: now also IC2.PH1(TXD2)
- net MISO: now also IC2.(MISO/PCINT3)PB3, J2.11, J3.DATA_OUT, J4.1; no longer J31.11, J6.DATA_OUT
- net MOSI: now also IC2.(MOSI/PCINT2)PB2, J3.DATA_IN, J4.4; no longer J6.DATA_IN
- net N$13: now also R10.1; no longer R3.1
- net SCK: now also IC2.(SCK/PCINT1)PB1, J2.12, J3.SCLK, J4.3; no longer J31.12, J6.SCLK
- net X_DIR: now also IC2.(OC3A/AIN1)PE3, J6.3; no longer J58.4
- net X_STEP: now also IC2.(OC0B)PG5, J6.4; no longer J58.3
- net X_VREF: now also IC2.(ADC0)PF0, J6.13; no longer J58.13
- net Y_DIR: now also IC2.PH4(OC4B), J6.5; no longer J58.6
- net Y_STEP: now also IC2.PH3(OC4A), J6.6; no longer J58.5
- net Y_VREF: now also IC2.(ADC1)PF1, J6.14; no longer J58.14
- net Z_DIR: now also IC2.(A13)PC5, J6.7; no longer J58.8
- net Z_STEP: now also IC2.(A14)PC6, J6.8; no longer J58.7
- net Z_VREF: now also IC2.(ADC2)PF2, J6.15; no longer J58.15
Other:
- note added: "3D Printer Controller - Microcontroller / Display board"
- note added: "FT230X"
- note removed: "3D Printer Controller - Input Power Distribution, High-Current Switches and Thermocouple Amplifiers"
- note removed: "Buzzer and Oscillator"
- note removed: "For driving fans, etc."
- note removed: "Rotary Encoder"
- moved on the sheet: C1, LCD1, LED1, R1, R12, R2, R3, VR1
