File: PololuStepperDriverCarrierBoard.brd (EAGLE design)
At the start: 106.7 x 50.8 mm, 42 parts, among them J1 MS1, J10 Y Stepper, J11 Interface, J12 MS1, J13 MS2, J14 A4988BREAKOUT, J15 MS3, J16 Z Stepper, J17 MS1, J18 24V Input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

Commit message: foo
Parts:
- removed J11: Interface, con-harting:CON20L
- added J28: Interface, con-harting:CON26L
- moved SY1 19.1 mm to (91.4, 5.08)
- moved J18 6.48 mm to (72.4, 7.62)
- moved F1 6.35 mm to (53.3, 6.35)
Connections:
- new net E1_EN: J20.EN, J28.21
- new net E2_EN: J25.EN, J28.22
- new net X_EN: J28.18, J3.EN
- new net Y_EN: J28.19, J8.EN
- new net Z_EN: J14.EN, J28.20
- net +24V: now also J28.24, J28.26; no longer J11.20
- net +3V3: now also J28.23, J28.25; no longer J11.18, J11.2
- net E1_DIR: now also J28.9; no longer J11.10
- net E1_STEP: now also J28.10; no longer J11.9
- net E1_VREF: now also J28.16; no longer J11.16
- net E2_DIR: now also J28.11; no longer J11.12
- net E2_STEP: now also J28.12; no longer J11.11
- net E2_VREF: now also J28.17; no longer J11.17
- net GND: now also J28.1, J28.2; no longer J11.1, J11.19
- net X_DIR: now also J28.3; no longer J11.4
- net X_STEP: now also J28.4; no longer J11.3
- net X_VREF: now also J28.13; no longer J11.13
- net Y_DIR: now also J28.5; no longer J11.6
- net Y_STEP: now also J28.6; no longer J11.5
- net Y_VREF: now also J28.14; no longer J11.14
- net Z_DIR: now also J28.7; no longer J11.8
- net Z_STEP: now also J28.8; no longer J11.7
- net Z_VREF: now also J28.15; no longer J11.15
Routing:
- net E2_EN: track 0.00 -> 61.6 mm, vias 0 -> 1
- net +3V3: track 212.9 -> 272.8 mm
- net E1_EN: track 0.00 -> 46.3 mm, vias 0 -> 1
- net X_EN: track 0.00 -> 33.3 mm
- net Z_EN: track 0.00 -> 25.0 mm, vias 0 -> 1
- net Y_EN: track 0.00 -> 19.4 mm, vias 0 -> 1
- net +24V: track 186.2 -> 198.7 mm
- net Z_DIR: track 53.2 -> 57.5 mm
- net Y_DIR: track 35.4 -> 39.8 mm
- net X_DIR: track 17.7 -> 22.0 mm
- net E2_DIR: track 88.0 -> 92.4 mm
- net E1_DIR: track 70.6 -> 75.0 mm
- net Z_STEP: track 55.0 -> 53.2 mm
- net Y_STEP: track 37.2 -> 35.4 mm
- net X_STEP: track 19.4 -> 17.7 mm
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